File: hardware/pcb.sch (EAGLE design)
At the start: 218 parts, among them IC1 LM386N-3, IC2 TL072P, IC6 7805

Commit message: PCB final (in production)
Parts:
- removed C11: 100n, rcl:C-EUC0805
- added C4: 100n, capacitor-wima:C5/3.5
- LED1, LED10, LED100, LED101, LED102, LED103, LED104, LED105, LED106, LED107, LED108, LED109, LED11, LED110, LED111, LED112, LED113, LED114, LED115, LED116, LED117, LED118, LED119, LED12, LED120, LED121, LED122, LED123, LED124, LED125, LED126, LED127, LED128, LED129, LED13, LED130, LED131, LED132, LED133, LED134, LED135, LED136, LED137, LED138, LED139, LED14, LED140, LED141, LED142, LED143, LED144, LED145, LED146, LED147, LED148, LED149, LED15, LED150, LED16, LED17, LED18, LED19, LED2, LED20, LED21, LED22, LED23, LED24, LED25, LED26, LED27, LED28, LED29, LED3, LED30, LED31, LED32, LED33, LED34, LED35, LED36, LED37, LED38, LED39, LED4, LED40, LED41, LED42, LED43, LED44, LED45, LED46, LED47, LED48, LED49, LED5, LED50, LED51, LED52, LED53, LED54, LED55, LED56, LED57, LED58, LED59, LED6, LED60, LED61, LED62, LED63, LED64, LED65, LED66, LED67, LED68, LED69, LED7, LED70, LED71, LED72, LED73, LED74, LED75, LED76, LED77, LED78, LED79, LED8, LED80, LED81, LED82, LED83, LED84, LED85, LED86, LED87, LED88, LED89, LED9, LED90, LED91, LED92, LED93, LED94, LED95, LED96, LED97, LED98, LED99: value (none) -> led 0805
- SPEAKER_SELECT: device switch:M9040P -> adafruit:EG1218S
- T1, T10, T2, T3, T4, T5, T6, T7, T8, T9: value (none) -> PNP SOT23
- renumbered JACK_INPUT to ADC_INPUT
Connections:
- net GND: now also C4.1; no longer C11.1
- net N$36: now also C4.2; no longer C11.2
